File: WifiRadio_firmware/Eagle/boombox_power_high_amp.sch (EAGLE design)
At the start: 7 parts, among them IC1 7805TV, J1 POWER_JACKPTH, Q1 MJE3055

Commit message: Modified boards, changed pin asignment in lcd driver
Parts:
- removed IC1: 7805TV, linear:7805TV
- removed JP1: (no value), pinhead:PINHD-1X2
- removed Q1: MJE3055, transistor-power:MJE3055
- added 5VOUT: (no value), pinhead:PINHD-1X2/90
- added IC2: 7805T, linear:7805T
- added LED1: (no value), led:LED3MM
- added Q2: BD243, transistor-npn:BD243
- added R1: 330R, resistor:R-EU_0309/V
Connections:
- new net N$1: J1.GNDBREAK
- new net N$3: LED1.C, R1.1
- net 9V: now also IC2.VI, Q2.C; no longer IC1.VI, Q1.C
- net GND: now also 5VOUT.2, IC2.GND, J1.GND, R1.2; no longer IC1.GND, J1.GNDBREAK, JP1.2
- net N$2: now also 5VOUT.1, LED1.A, Q2.E; no longer JP1.1, Q1.E
- net VCC: now also IC2.VO, Q2.B; no longer IC1.VO, Q1.B
Changed lines of the file:
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@@
 <part name="J1" library="SparkFun" deviceset="POWER_JACK" device="PTH"/>
 <part name="S1" library="SparkFun" deviceset="SWITCH-SPST" device="PTH"/>
-<part name="JP1" library="pinhead" deviceset="PINHD-1X2" device=""/>
-<part name="Q1" library="transistor-power" deviceset="MJE3055" device=""/>
-<part name="IC1" library="linear" deviceset="78*" device="TV" technology="05"/>
 <part name="C1" library="SparkFun" deviceset="CAP_POL" device="PTH4" value="2200uF"/>
 <part name="C2" library="SparkFun" deviceset="CAP_POL" device="PTH4" value="2200uF"/>
@@
 <part name="GND4" library="SparkFun" deviceset="GND" device=""/>
 <part name="GND1" library="SparkFun" deviceset="GND" device=""/>
+<part name="5VOUT" library="pinhead" deviceset="PINHD-1X2" device="/90"/>
+<part name="LED1" library="led" deviceset="LED" device="3MM"/>
+<part name="R1" library="resistor" deviceset="R-EU_" device="0309/V" value="330R"/>
+<part name="Q2" library="transistor-npn" deviceset="BD243*" device=""/>
+<part name="IC2" library="linear" deviceset="78*" device="T" technology="05"/>
 </parts>
 <sheets>
@@
 <instance part="J1" gate="G$1" x="-15.24" y="114.3"/>
 <instance part="S1" gate="1" x="-7.62" y="124.46"/>
-<instance part="JP1" gate="G$1" x="53.34" y="106.68"/>
-<instance part="Q1" gate="1" x="30.48" y="116.84"/>
-<instance part="IC1" gate="A1" x="15.24" y="121.92"/>
 <instance part="C1" gate="G$1" x="0" y="114.3"/>
 <instance part="C2" gate="G$1" x="33.02" y="109.22"/>
 <instance part="GND3" gate="1" x="15.24" y="106.68"/>
 <instance part="GND4" gate="1" x="33.02" y="101.6"/>
-<instance part="GND1" gate="1" x="50.8" y="101.6"/>
+<instance part="GND1" gate="1" x="55.88" y="124.46" rot="R180"/>
+<instance part="5VOUT" gate="G$1" x="53.34" y="114.3" rot="R180"/>
+<instance part="LED1" gate="G$1" x="43.18" y="114.3" rot="R180"/>
+<instance part="R1" gate="G$1" x="50.8" y="121.92"/>
+<instance part="Q2" gate="G$1" x="30.48" y="116.84"/>
+<instance part="IC2" gate="A1" x="15.24" y="121.92"/>
 </instances>
 <busses>
@@
 <segment>
 <label x="40.64" y="121.92" size="1.778" layer="95"/>
-<pinref part="Q1" gate="1" pin="B"/>
 <wire x1="27.94" y1="121.92" x2="27.94" y2="116.84" width="0.1524" layer="91"/>
-<pinref part="IC1" gate="A1" pin="VO"/>
+<wire x1="27.94" y1="121.92" x2="25.4" y2="121.92" width="0.1524" layer="91"/>
+<pinref part="Q2" gate="G$1" pin="B"/>
+<junction x="27.94" y="116.84"/>
+<pinref part="IC2" gate="A1" pin="VO"/>
 <wire x1="25.4" y1="121.92" x2="22.86" y2="121.92" width="0.1524" layer="91"/>
-<wire x1="27.94" y1="121.92" x2="25.4" y2="121.92" width="0.1524" layer="91"/>
 <junction x="25.4" y="121.92"/>
 </segment>
@@
 <wire x1="-7.62" y1="104.14" x2="-7.62" y2="101.6" width="0.1524" layer="91"/>
 <junction x="-7.62" y="104.14"/>
-<pinref part="J1" gate="G$1" pin="GNDBREAK"/>
-<wire x1="-12.7" y1="119.38" x2="-10.16" y2="119.38" width="0.1524" layer="91"/>
-<wire x1="-10.16" y1="119.38" x2="-10.16" y2="114.3" width="0.1524" layer="91"/>
-<junction x="-12.7" y="119.38"/>
+<pinref part="J1" gate="G$1" pin="GND"/>
+<wire x1="-10.16" y1="116.84" x2="-10.16" y2="114.3" width="0.1524" layer="91"/>
+<wire x1="-10.16" y1="116.84" x2="-12.7" y2="116.84" width="0.1524" layer="91"/>
+<junction x="-12.7" y="116.84"/>
 </segment>
 <segment>
@@
 <wire x1="0" y1="109.22" x2="15.24" y2="109.22" width="0.1524" layer="91"/>
 <wire x1="15.24" y1="116.84" x2="15.24" y2="114.3" width="0.1524" layer="91"/>
-<pinref part="IC1" gate="A1" pin="GND"/>
+<junction x="15.24" y="109.22"/>
+<pinref part="IC2" gate="A1" pin="GND"/>
 <wire x1="15.24" y1="114.3" x2="15.24" y2="109.22" width="0.1524" layer="91"/>
-<junction x="15.24" y="109.22"/>
 <junction x="15.24" y="114.3"/>
 </segment>
@@
 <pinref part="C2" gate="G$1" pin="-"/>
 <pinref part="GND4" gate="1" pin="GND"/>
+<junction x="33.02" y="104.14"/>
 </segment>
 <segment>
-<pinref part="JP1" gate="G$1" pin="2"/>
 <pinref part="GND1" gate="1" pin="GND"/>
-<wire x1="50.8" y1="104.14" x2="50.8" y2="106.68" width="0.1524" layer="91"/>
+<pinref part="R1" gate="G$1" pin="2"/>
+<pinref part="5VOUT" gate="G$1" pin="2"/>
+<wire x1="55.88" y1="114.3" x2="55.88" y2="121.92" width="0.1524" layer="91"/>
+<junction x="55.88" y="121.92"/>
+<junction x="55.88" y="114.3"/>
 </segment>
 </net>
@@
 <junction x="-2.54" y="121.92"/>
 <wire x1="7.62" y1="121.92" x2="5.08" y2="121.92" width="0.1524" layer="91"/>
-<pinref part="IC1" gate="A1" pin="VI"/>
 <junction x="5.08" y="121.92"/>
 <wire x1="5.08" y1="121.92" x2="0" y2="121.92" width="0.1524" layer="91"/>
 <wire x1="5.08" y1="121.92" x2="5.08" y2="127" width="0.1524" layer="91"/>
 <wire x1="5.08" y1="127" x2="33.02" y2="127" width="0.1524" layer="91"/>
-<pinref part="Q1" gate="1" pin="C"/>
 <wire x1="33.02" y1="127" x2="33.02" y2="121.92" width="0.1524" layer="91"/>
 <pinref part="C1" gate="G$1" pin="+"/>
 <junction x="0" y="121.92"/>
+<pinref part="Q2" gate="G$1" pin="C"/>
+<junction x="33.02" y="121.92"/>
+<pinref part="IC2" gate="A1" pin="VI"/>
 </segment>
 </net>
-<net name="N$1" class="0">
+<net name="N$5" class="0">
 <segment>
 <pinref part="S1" gate="1" pin="P"/>
@@
 <net name="N$2" class="0">
 <segment>
-<pinref part="Q1" gate="1" pin="E"/>
 <pinref part="C2" gate="G$1" pin="+"/>
-<pinref part="JP1" gate="G$1" pin="1"/>
-<wire x1="33.02" y1="111.76" x2="50.8" y2="111.76" width="0.1524" layer="91"/>
-<wire x1="50.8" y1="111.76" x2="50.8" y2="109.22" width="0.1524" layer="91"/>
+<pinref part="LED1" gate="G$1" pin="A"/>
+<wire x1="43.18" y1="111.76" x2="33.02" y2="111.76" width="0.1524" layer="91"/>
+<pinref part="Q2" gate="G$1" pin="E"/>
 <junction x="33.02" y="111.76"/>
+<pinref part="5VOUT" gate="G$1" pin="1"/>
+<wire x1="55.88" y1="111.76" x2="43.18" y2="111.76" width="0.1524" layer="91"/>
+<junction x="43.18" y="111.76"/>
+<junction x="55.88" y="111.76"/>
 </segment>
 </net>
+<net name="N$3" class="0">
+<segment>
+<pinref part="LED1" gate="G$1" pin="C"/>
+<wire x1="43.18" y1="119.38" x2="43.18" y2="121.92" width="0.1524" layer="91"/>
+<pinref part="R1" gate="G$1" pin="1"/>
+<wire x1="43.18" y1="121.92" x2="45.72" y2="121.92" width="0.1524" layer="91"/>
+<junction x="45.72" y="121.92"/>
+</segment>
+</net>
+<net name="N$1" class="0">
+<segment>
+<pinref part="J1" gate="G$1" pin="GNDBREAK"/>
+<wire x1="-12.7" y1="119.38" x2="-10.16" y2="119.38" width="0.1524" layer="91"/>
+<junction x="-12.7" y="119.38"/>
+</segment>
+</net>
